File: Hardware/Qwiic 1x1/SparkFun_Qwiic_6DoF_BMI270.sch (EAGLE design)
At the start: 29 parts, among them J1 QWIIC_RIGHT_ANGLE, J2 QWIIC_RIGHT_ANGLE, U1 BMI270

Commit message: Checklist updates
Change max VDD to VDD range
Add ordering instructions
Add axis labels to bottom silk
Add silk label to power LED
Other:
- note added: "VDD Range: 1.71V - 3.6V"
- note removed: "Max voltage: 3.6V"
Changed lines of the file:
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@@
 <text x="73.66" y="75.946" size="1.778" layer="97" font="vector" align="center">Cut I2C jumper to
 remove pullup resistors</text>
-<text x="73.66" y="159.766" size="1.778" layer="97" font="vector" align="center">Max voltage: 3.6V</text>
+<text x="73.66" y="159.766" size="1.778" layer="97" font="vector" align="center">VDD Range:
+1.71V - 3.6V</text>
 <wire x1="73.66" y1="68.58" x2="0" y2="68.58" width="0.1524" layer="97" style="longdash"/>
 <wire x1="73.66" y1="68.58" x2="73.66" y2="0" width="0.1524" layer="97" style="longdash"/>
@@
 </instance>
 <instance part="ADR" gate="G$1" x="111.76" y="30.48" smashed="yes" rot="MR0">
-<attribute name="NAME" x="106.68" y="30.48" size="1.778" layer="95" font="vector" rot="MR0" align="center"/>
+<attribute name="NAME" x="108.712" y="30.48" size="1.778" layer="95" font="vector" rot="MR270" align="center"/>
 </instance>
 <instance part="SUPPLY3" gate="G$1" x="111.76" y="50.8" smashed="yes">

Commit message: Add "default" to I2C address in schematics
Other:
- note added: "(Default) GND: 0x68 3.3V: 0x69 Open: SPI"
- note removed: "GND: 0x68 3.3V: 0x69 Open: SPI"
Changed lines of the file:
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@@
 <sheet>
 <plain>
-<text x="101.6" y="30.48" size="1.778" layer="97" font="vector" align="center-right">GND: 0x68
+<text x="101.6" y="30.48" size="1.778" layer="97" font="vector" align="center-right">(Default) GND: 0x68
 3.3V: 0x69
 Open: SPI</text>

Commit message: Remove PROD_ID from headers of 1x1
Parts:
- J3, J4: device SparkFun-Connectors:CONN_06NO_SILK_FEMALE_PTH -> SparkFun-Connectors:CONN_06NO_SILK_NO_POP
Changed lines of the file:
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@@
 <part name="SUPPLY4" library="SparkFun-PowerSymbols" deviceset="3.3V" device=""/>
 <part name="J1" library="SparkFun-Connectors" deviceset="QWIIC_CONNECTOR" device="JS-1MM" value="QWIIC_RIGHT_ANGLE"/>
-<part name="J3" library="SparkFun-Connectors" deviceset="CONN_06" device="NO_SILK_FEMALE_PTH"/>
+<part name="J3" library="SparkFun-Connectors" deviceset="CONN_06" device="NO_SILK_NO_POP"/>
 <part name="SUPPLY5" library="SparkFun-PowerSymbols" deviceset="3.3V" device=""/>
 <part name="GND4" library="SparkFun-PowerSymbols" deviceset="GND" device=""/>
@@
 <part name="R6" library="SparkFun-Resistors" deviceset="100KOHM" device="-0603-1/10W-1%" value="100k"/>
 <part name="SUPPLY9" library="SparkFun-PowerSymbols" deviceset="3.3V" device=""/>
-<part name="J4" library="SparkFun-Connectors" deviceset="CONN_06" device="NO_SILK_FEMALE_PTH"/>
+<part name="J4" library="SparkFun-Connectors" deviceset="CONN_06" device="NO_SILK_NO_POP"/>
 <part name="C2" library="SparkFun-Capacitors" deviceset="0.1UF" device="-0603-25V-(+80/-20%)" value="0.1uF"/>
 <part name="SUPPLY10" library="SparkFun-PowerSymbols" deviceset="3.3V" device=""/>
